Commit message: stlを使わないurdfの作成とstlを使ったurdfの作成

File: r5sr_description/urdf/r5sr_arm_simple.urdf (robot description, URDF)
Before this commit: robot r5sr, 8 links, 7 joints
Links:
- link body0_link_yaw: geometry visual box size=0.1 0.1 0.02
- link body1_link: geometry visual box size=0.1 0.2 0.04
- link body2_link: geometry visual box size=0.55 0.1 0.04
- link body3_link: geometry visual box size=0.55 0.1 0.03
- link body4_link: geometry visual box size=0.045 0.045 0.045
- link body5_link: geometry visual box size=0.06 0.03 0.03
- link body6_link: geometry visual box size=0.03 0.06 0.03
Joints:
- joint body6_joint: origin xyz=0.05 0 0.033 rpy=0 0 0 -> xyz=0.042 0 0 rpy=0 0 0
