Commit message: moveit2用のパッケージを作成（未動作）
https://zenn.dev/tasada038/articles/940ef193a4a28a
これ通りにxacroのファイルを置いて、diplay.launchでジョイントを動かせるようになった。moveit2はまだ動かせてない

File: r5sr_description/urdf/r5sr_arm.urdf (robot description, URDF)
Before this commit: robot r5sr, 8 links, 7 joints
Links:
- link body0_link_yaw: geometry visual mesh filename=package://r5sr_description/meshes/arm_parts_0.stl
- link body1_link: geometry visual mesh filename=package://r5sr_description/meshes/arm_parts_1.stl
- link body2_link: geometry visual mesh filename=package://r5sr_description/meshes/arm_parts_2.stl
- link body3_link: geometry visual mesh filename=package://r5sr_description/meshes/arm_parts_3.stl
- link body4_link: geometry visual mesh filename=package://r5sr_description/meshes/arm_parts_4.stl
- link body5_link: geometry visual mesh filename=package://r5sr_description/meshes/arm_parts_5.stl
- link body6_link: geometry visual mesh filename=package://r5sr_description/meshes/arm_parts_6.stl
