Commit message: 俯瞰アーム xacro作成

File: r5sr_description/urdf/materials.xacro (robot description, xacro)
@@ -4,6 +4,9 @@
    <color rgba="1 1 1 1"/>
   </material>
-  <material name="blue">
+  <material name="red">
     <color rgba="0.8 0 0 1"/>
   </material>
+  <material name="green">
+    <color rgba="0 0.8 0 1"/>
+  </material>
 </robot>

File: r5sr_description/urdf/r5sr.xacro (robot description, xacro)
@@ -4,5 +4,5 @@
 <xacro:include filename="$(find r5sr_description)/urdf/r5sr.trans" />
 <xacro:include filename="$(find r5sr_description)/urdf/r5sr_description.xacro" />
-<xacro:r5sr_description main_color="blue" sub_color="white" />
+<xacro:r5sr_description main_color="red" sub_color1="white" sub_color2="green" />
 <!-- Import Robot ros2_control description -->
 <xacro:include filename="$(find r5sr_description)/ros2_control/r5sr_ros2_control.xacro" />

File: r5sr_description/urdf/r5sr_description.xacro (robot description, xacro)
@@ -1,5 +1,5 @@
 <?xml version="1.0" ?>
 <robot name="r5sr" xmlns:xacro="http://www.ros.org/wiki/xacro" >
-  <xacro:macro name="r5sr_description" params="main_color sub_color">
+  <xacro:macro name="r5sr_description" params="main_color sub_color1 sub_color2">
     <link name="base_link">
         <visual>
@@ -16,5 +16,5 @@
         </geometry>
         <origin xyz="0 0 0" rpy="0 0 0"/>
-        <material name="${sub_color}"/>
+        <material name="${sub_color1}"/>
         </visual>
     </link>
@@ -55,4 +55,31 @@
         </visual>
     </link>
+    <link name="vision_arm_body1_link">
+        <visual>
+        <geometry>
+            <cylinder length="0.6" radius="0.01"/>
+        </geometry>
+        <origin xyz="0 0 0.3" rpy="0 0 0"/>
+        <material name="${sub_color1}"/>
+        </visual>
+    </link>
+    <link name="vision_arm_body2_link">
+        <visual>
+        <geometry>
+            <box size="0.04 0.04 0.02"/>
+        </geometry>
+        <origin xyz="0 0 0" rpy="0 0 0"/>
+        <material name="${main_color}"/>
+        </visual>
+    </link>
+    <link name="vision_arm_body3_link">
+        <visual>
+        <geometry>
+            <box size="0.05 0.02 0.02"/>
+        </geometry>
+        <origin xyz="0.02 0 0" rpy="0 0 0"/>
+        <material name="${sub_color2}"/>
+        </visual>
+    </link>
     <link name="body5_link">
         <visual>
@@ -70,5 +97,5 @@
         </geometry>
         <origin xyz="-0.175 0 -0.22" rpy="0 0 0"/>
-        <material name="${sub_color}"/>
+        <material name="${sub_color1}"/>
         </visual>
     </link>
@@ -122,4 +149,25 @@
         <limit lower="-3.14159265" upper="3.14159265" effort="0" velocity="3.1415"/>
     </joint>
+    <joint name="vision_arm_body1_joint" type="revolute">
+        <parent link="body4_link"/>
+        <child  link="vision_arm_body1_link"/>
+        <axis xyz="0 1 0"/>
+        <origin xyz="0 0.08 0" rpy="0 -1.57075 0"/>
+        <limit lower="-3.15" upper="3.15" effort="0" velocity="3.1415"/>
+    </joint>
+    <joint name="vision_arm_body2_joint" type="revolute">
+        <parent link="vision_arm_body1_link"/>
+        <child  link="vision_arm_body2_link"/>
+        <axis xyz="0 1 0"/>
+        <origin xyz="0 -0.03 0.6" rpy="1.57075 1.57075 1.57075"/>
+        <limit lower="-3.15" upper="3.15" effort="0" velocity="3.1415"/>
+    </joint>
+    <joint name="vision_arm_body3_joint" type="revolute">
+        <parent link="vision_arm_body2_link"/>
+        <child  link="vision_arm_body3_link"/>
+        <axis xyz="0 0 1"/>
+        <origin xyz="0 0 0.02" rpy="0 0 0"/>
+        <limit lower="-3.15" upper="3.15" effort="0" velocity="3.1415"/>
+    </joint>
   </xacro:macro>
 </robot>
