Commit message: 実機で動作した！

File: r5sr_description/urdf/r5sr_description.xacro (robot description, xacro)
@@ -112,5 +112,5 @@
         <axis xyz="0 0 1"/>
         <origin xyz="0 0 0" rpy="0 0 0"/>
-        <limit lower="-1.575" upper="1.575" effort="0" velocity="3.1415"/>
+        <limit lower="-3.1415" upper="3.1415" effort="0" velocity="3.1415"/>
     </joint>
     <joint name="body2_joint" type="revolute">
@@ -119,5 +119,5 @@
         <axis xyz="0 1 0"/>
         <origin xyz="0 0 0.101" rpy="0 0 0"/>
-        <limit lower="-0" upper="3.15" effort="0" velocity="3.1415"/>
+        <limit lower="-3.1415" upper="3.1415" effort="0" velocity="3.1415"/>
     </joint>
     <joint name="body3_joint" type="revolute">
@@ -126,5 +126,5 @@
         <axis xyz="0 1 0"/>
         <origin xyz="-0.480 -0. 0" rpy="0 0 0"/>
-        <limit lower="-3.15" upper="0" effort="0" velocity="3.1415"/>
+        <limit lower="-3.1415" upper="3.1415" effort="0" velocity="3.1415"/>
     </joint>
         <joint name="body4_joint" type="revolute">
@@ -133,5 +133,5 @@
         <axis xyz="0 1 0"/>
         <origin xyz="0.56235 0 0.0443" rpy="0 0 0"/>
-        <limit lower="-3.15" upper="3.15" effort="0" velocity="3.1415"/>
+        <limit lower="-3.1415" upper="3.1415" effort="0" velocity="3.1415"/>
     </joint>
     <joint name="body5_joint" type="revolute">
@@ -140,5 +140,5 @@
         <axis xyz="0 0 1"/>
         <origin xyz="0.042 0 0.045" rpy="0 0 0"/>
-        <limit lower="-3.15" upper="3.15" effort="0" velocity="3.1415"/>
+        <limit lower="-3.1415" upper="3.1415" effort="0" velocity="3.1415"/>
     </joint>
     <joint name="body6_joint" type="revolute">
@@ -147,5 +147,5 @@
         <axis xyz="1 0 0"/>
         <origin xyz="0.05 0 0.033" rpy="0 0 0"/>
-        <limit lower="-3.14159265" upper="3.14159265" effort="0" velocity="3.1415"/>
+        <limit lower="-3.1415" upper="3.1415" effort="0" velocity="3.1415"/>
     </joint>
     <joint name="vision_arm_body1_joint" type="revolute">
@@ -154,5 +154,5 @@
         <axis xyz="0 1 0"/>
         <origin xyz="0 0.08 0" rpy="0 -1.57075 0"/>
-        <limit lower="-3.15" upper="3.15" effort="0" velocity="3.1415"/>
+        <limit lower="-3.1415" upper="3.1415" effort="0" velocity="3.1415"/>
     </joint>
     <joint name="vision_arm_body2_joint" type="revolute">
@@ -161,5 +161,5 @@
         <axis xyz="0 1 0"/>
         <origin xyz="0 -0.03 0.6" rpy="1.57075 1.57075 1.57075"/>
-        <limit lower="-3.15" upper="3.15" effort="0" velocity="3.1415"/>
+        <limit lower="-3.1415" upper="3.1415" effort="0" velocity="3.1415"/>
     </joint>
     <joint name="vision_arm_body3_joint" type="revolute">
@@ -168,5 +168,5 @@
         <axis xyz="0 0 1"/>
         <origin xyz="0 0 0.02" rpy="0 0 0"/>
-        <limit lower="-3.15" upper="3.15" effort="0" velocity="3.1415"/>
+        <limit lower="-3.1415" upper="3.1415" effort="0" velocity="3.1415"/>
     </joint>
   </xacro:macro>
