Commit message: servo teleopの実行ファイル作った(未動作)
動かそうとすると、定義していないpanda_link1（demo用のロボットの関節名）がurdf上にないと警告が出て、全く動作させることができない。
issueにも同じような人がいる。
https://github.com/ros-planning/moveit2/issues/1194

File: r5sr_description/ros2_control/r5sr_ros2_control.xacro (robot description, xacro)
@@ -1,5 +1,6 @@
 <?xml version="1.0" ?>
 <robot name="r5sr" xmlns:xacro="http://www.ros.org/wiki/xacro" >
-  <xacro:macro name="r5sr_ros2_control" params="name">
+  <xacro:macro name="r5sr_ros2_control" params="name initial_positions_file">
+    <xacro:property name="initial_positions" value="${load_yaml(initial_positions_file)['initial_positions']}"/>
     <!-- Connect GazeboSystem -->>
     <ros2_control name="${name}" type="system">
@@ -19,4 +20,5 @@
       </joint>
       <joint name="body1_joint">
+        <param name="initial_position">${initial_positions['body1_joint']}</param>
         <command_interface name="position">
           <param name="min">-3.15</param>
@@ -29,4 +31,5 @@
       </joint>
       <joint name="body2_joint">
+        <param name="initial_position">${initial_positions['body2_joint']}</param>
         <command_interface name="position">
           <param name="min">-3.15</param>
@@ -39,4 +42,5 @@
       </joint>
       <joint name="body3_joint">
+        <param name="initial_position">${initial_positions['body3_joint']}</param>
         <command_interface name="position">
           <param name="min">-3.15</param>
@@ -49,4 +53,5 @@
       </joint>
       <joint name="body4_joint">
+        <param name="initial_position">${initial_positions['body4_joint']}</param>
         <command_interface name="position">
           <param name="min">-3.15</param>
@@ -59,4 +64,5 @@
       </joint>
       <joint name="body5_joint">
+        <param name="initial_position">${initial_positions['body5_joint']}</param>
         <command_interface name="position">
           <param name="min">-3.15</param>
@@ -69,4 +75,5 @@
       </joint>
       <joint name="body6_joint">
+        <param name="initial_position">${initial_positions['body6_joint']}</param>
         <command_interface name="position">
           <param name="min">-3.15</param>

File: r5sr_description/urdf/r5sr.xacro (robot description, xacro)
@@ -7,4 +7,4 @@
 <!-- Import Robot ros2_control description -->
 <xacro:include filename="$(find r5sr_description)/ros2_control/r5sr_ros2_control.xacro" />
-<xacro:r5sr_ros2_control name="r5sr" />
+<xacro:r5sr_ros2_control name="r5sr" initial_positions_file="$(find r5sr_moveit_config)/config/initial_positions.yaml" />
 </robot>

Commit message: #13:俯瞰アーム追加パッケージ完成
動作確認したつもり

File: r5sr_description/ros2_control/r5sr_ros2_control.xacro (robot description, xacro)
@@ -85,4 +85,37 @@
         <state_interface name="velocity"/>
       </joint>
+      <joint name="vision_arm_body1_joint">
+        <param name="initial_position">${initial_positions['vision_arm_body1_joint']}</param>
+        <command_interface name="position">
+          <param name="min">-3.15</param>
+          <param name="max">3.15</param>
+        </command_interface>
+        <state_interface name="position">
+          <param name="initial_value">0.0</param>
+        </state_interface>
+        <state_interface name="velocity"/>
+      </joint>
+      <joint name="vision_arm_body2_joint">
+        <param name="initial_position">${initial_positions['vision_arm_body2_joint']}</param>
+        <command_interface name="position">
+          <param name="min">-3.15</param>
+          <param name="max">3.15</param>
+        </command_interface>
+        <state_interface name="position">
+          <param name="initial_value">0.0</param>
+        </state_interface>
+        <state_interface name="velocity"/>
+      </joint>
+      <joint name="vision_arm_body3_joint">
+        <param name="initial_position">${initial_positions['vision_arm_body3_joint']}</param>
+        <command_interface name="position">
+          <param name="min">-3.15</param>
+          <param name="max">3.15</param>
+        </command_interface>
+        <state_interface name="position">
+          <param name="initial_value">0.0</param>
+        </state_interface>
+        <state_interface name="velocity"/>
+      </joint>
     </ros2_control>
   </xacro:macro>

File: r5sr_description/urdf/r5sr.xacro (robot description, xacro)
@@ -6,5 +6,5 @@
 <xacro:r5sr_description main_color="red" sub_color1="white" sub_color2="green" />
 <!-- Import Robot ros2_control description -->
-<xacro:include filename="$(find r5sr_description)/ros2_control/r5sr_ros2_control.xacro" />
+<xacro:include filename="$(find r5sr_description)/ros2_control/r5sr_ros2_control.xacro" /> -->
 <xacro:r5sr_ros2_control name="r5sr" initial_positions_file="$(find r5sr_moveit_config)/config/initial_positions.yaml" />
 </robot>
