Commit message: fix justfile

File: src/r5sr_moveit_config/config/r5sr.ros2_control.xacro (robot description, xacro)
@@ -64,4 +64,18 @@
                 <state_interface name="velocity"/>
             </joint>
+            <joint name="crawler_left_joint">
+                <command_interface name="position"/>
+                <state_interface name="position">
+                  <param name="initial_value">${initial_positions['crawler_left_joint']}</param>
+                </state_interface>
+                <state_interface name="velocity"/>
+            </joint>
+            <joint name="crawler_right_joint">
+                <command_interface name="position"/>
+                <state_interface name="position">
+                  <param name="initial_value">${initial_positions['crawler_right_joint']}</param>
+                </state_interface>
+                <state_interface name="velocity"/>
+            </joint>
             <joint name="overhead_wrist_pitch_joint">
                 <command_interface name="position"/>
