Commit message: lidarslamで動作かくにん

File: src/r5sr_description/urdf/r5sr.xacro (robot description, xacro)
@@ -279,4 +279,10 @@
         </joint>
         <link name="fisheye_front_link" />
+        <joint name="mid360_joint" type="fixed">
+            <parent link="forearm_link" />
+            <child link="mid360" />
+            <origin xyz="0.25 0 0.07" rpy="0 0.1 3.14159" />
+        </joint>
+        <link name="mid360" />
         <!-- others -->
         <joint name="base_footprint_joint" type="fixed">

Commit message: camerainfo調整

File: src/r5sr_description/urdf/r5sr.xacro (robot description, xacro)
@@ -252,5 +252,5 @@
             <parent link="end_effector_link" />
             <child link="hand_camera_link" />
-            <origin xyz="0.05 0 0" rpy="0 0 0" />
+            <origin xyz="0.05 0 0" rpy="-1.57079632679 0 -1.57079632679" />
         </joint>
         <link name="hand_camera_link" />
@@ -264,5 +264,5 @@
             <parent link="overhead_wrist_2_link" />
             <child link="vision_front_link" />
-            <origin xyz="0.03 0 0.001" rpy="0 0.1 0" />
+            <origin xyz="0.03 0 0.001" rpy="-1.57079632679 0 -1.57079632679" />
         </joint>
         <link name="vision_front_link" />

Commit message: camera調整

File: src/r5sr_description/urdf/r5sr.xacro (robot description, xacro)
@@ -270,5 +270,5 @@
             <parent link="overhead_wrist_2_link" />
             <child link="vision_rear_link" />
-            <origin xyz="-0.01 0 -0.001" rpy="3.1415 -0.5 0" />
+            <origin xyz="-0.01 0 -0.001" rpy="0 3.141592 -1.57079632679" />
         </joint>
         <link name="vision_rear_link" />
